File: schematic/schematic.sch (KiCad schematic (older format))
At the start: 5 parts, among them U1 LM7805_TO220

Commit message: Created schematic for the hardware of the project
Parts:
- removed U1: LM7805_TO220, TO_SOT_Packages_THT:TO-220_Vertical, symbol LM7805_TO220
- added A?: Arduino_Nano_v3.x, Modules:Arduino_Nano, symbol Arduino_Nano_v3.x
- added BT? (x3): Battery_Cell, symbol Battery_Cell
- added C? (x2): 100nF, symbol C
- added C?: 100uF, symbol CP
- added D? (x2): D_Schottky, symbol D_Schottky
- added D? (x2): D_Zener, symbol D_Zener
- added F? (x3): Fuse, symbol Fuse
- added J? (x2): Conn_01x01_Female, symbol Conn_01x01_Female
- added J?: Raspberry_Pi_2_3, Pin_Headers:Pin_Header_Straight_2x20, symbol Raspberry_Pi_2_3
- added JOY? (x2): KY-023, symbol KY-023
- added LM?: LM2587, fuse, symbol LM2587
- added M? (x2): Motor_DC, symbol Motor_DC
- added R? (x4): 10k, symbol R
- added SW?: SW_DIP_x01, symbol SW_DIP_x01
- added U?: Consider for stable powerLM7805_TO220, TO_SOT_Packages_THT:TO-220_Vertical, symbol LM7805_TO220
- added U?: L298(H)N, TO_SOT_Packages_THT:Multiwatt_15_Vertical, symbol L298(H)N
- added U?: ESP-12F, symbol ESP-12F
- added U?: MCP3204, symbol MCP3204
Connections:
- net labels removed: +12V
- wire segments 12 -> 136
- no-connect marks 0 -> 1
Other:
- moved on the sheet: C1, C2, C3, C4
